File: eagle/v1-controller.brd (EAGLE design)
At the start: 66 x 40.6 mm, 13 parts, among them Q1 DHT##, X1 RJ45-6L21-B

Commit message: Finished v1
Parts:
- removed U$1: RS485-ADAPTER, serge:RS485-ADAPTOR
- added Q2: RS485-ADAPTER0.05-CONNECTOR, serge:RS485-ADAPTOR-05
Connections:
- net D2: now also Q2.RE/DE; no longer U$1.RE/DE
- net GND: now also Q2.GND; no longer U$1.GND
- net N$5: now also Q2.12V-IN; no longer U$1.12V-IN
- net N$7: now also Q2.B; no longer U$1.B
- net N$8: now also Q2.A; no longer U$1.A
- net RX: now also Q2.RX; no longer U$1.RX
- net TX: now also Q2.TX; no longer U$1.TX
- net V+: now also Q2.12V-OUT; no longer U$1.12V-OUT
- net VCC: now also Q2.5V-IN; no longer U$1.5V-IN
Routing:
- net V+: track 3.96 -> 5.61 mm
- net N$7: track 22.5 -> 21.3 mm
- net D2: track 15.5 -> 14.3 mm
- net N$8: track 25.8 -> 24.7 mm
- net N$5: track 57.4 -> 56.4 mm
- net TX: track 8.89 -> 8.15 mm
- net RX: track 6.24 -> 5.61 mm
Changed lines of the file:
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@@
 <elements>
 <element name="U$2" library="serge" package="ARDUINO-PRO-MINI" value="ARDUINO-PRO-MINI" x="25.4" y="30.48" rot="R180"/>
-<element name="U$1" library="serge" package="RS485-ADAPTOR" value="RS485-ADAPTER" x="25.4" y="32.385"/>
 <element name="X1" library="con-tycoelectronics" package="RJ45-SHIELD1" value="RJ45-6L21-B" x="60.96" y="25.4" rot="R90">
 <attribute name="OC_NEWARK" value="unknown" x="60.96" y="25.4" size="1.778" layer="27" rot="R90" display="off"/>
@@
 <attribute name="OC_FARNELL" value="unknown" x="64.77" y="17.78" size="1.778" layer="27" rot="R180" display="off"/>
 </element>
+<element name="Q2" library="serge" package="RS485-ADAPTOR-05" value="RS485-ADAPTER0.05-CONNECTOR" x="24.13" y="30.48"/>
 </elements>
 <signals>
 <signal name="D2">
 <contactref element="U$2" pad="D2"/>
-<contactref element="U$1" pad="RE/DE"/>
-<wire x1="12.7" y1="31.623" x2="14.097" y2="31.623" width="0.4064" layer="16"/>
-<wire x1="14.097" y1="31.623" x2="15.24" y2="30.48" width="0.4064" layer="16"/>
-<wire x1="15.24" y1="30.48" x2="15.24" y2="26.035" width="0.4064" layer="16"/>
+<wire x1="15.24" y1="29.21" x2="15.24" y2="26.035" width="0.4064" layer="16"/>
 <wire x1="15.24" y1="26.035" x2="16.51" y2="24.765" width="0.4064" layer="16"/>
 <wire x1="16.51" y1="24.765" x2="20.32" y2="24.765" width="0.4064" layer="16"/>
 <wire x1="20.32" y1="24.765" x2="21.59" y2="23.495" width="0.4064" layer="16"/>
 <wire x1="21.59" y1="23.495" x2="21.59" y2="22.86" width="0.4064" layer="16"/>
+<contactref element="Q2" pad="RE/DE"/>
+<wire x1="12.7" y1="30.48" x2="13.97" y2="30.48" width="0.4064" layer="16"/>
+<wire x1="13.97" y1="30.48" x2="15.24" y2="29.21" width="0.4064" layer="16"/>
 </signal>
 <signal name="RX">
 <contactref element="U$2" pad="RX1"/>
 <contactref element="U$2" pad="RX2"/>
-<contactref element="U$1" pad="RX"/>
-<wire x1="12.7" y1="28.575" x2="12.7" y2="24.13" width="0.4064" layer="16"/>
 <wire x1="12.7" y1="24.13" x2="13.97" y2="22.86" width="0.4064" layer="16"/>
-<wire x1="12.7" y1="28.575" x2="8.89" y2="31.75" width="0" layer="19" extent="1-1"/>
+<contactref element="Q2" pad="RX"/>
+<wire x1="12.7" y1="27.94" x2="12.7" y2="24.13" width="0.4064" layer="16"/>
+<wire x1="12.7" y1="27.94" x2="8.89" y2="31.75" width="0" layer="19" extent="1-1"/>
 </signal>
 <signal name="TX">
 <contactref element="U$2" pad="TX1"/>
 <contactref element="U$2" pad="TX2"/>
-<contactref element="U$1" pad="TX"/>
-<wire x1="12.7" y1="30.099" x2="11.684" y2="30.099" width="0.4064" layer="16"/>
-<wire x1="11.684" y1="30.099" x2="10.795" y2="29.21" width="0.4064" layer="16"/>
-<wire x1="10.795" y1="29.21" x2="10.795" y2="23.495" width="0.4064" layer="16"/>
+<wire x1="10.795" y1="28.575" x2="10.795" y2="23.495" width="0.4064" layer="16"/>
 <wire x1="10.795" y1="23.495" x2="11.43" y2="22.86" width="0.4064" layer="16"/>
-<wire x1="11.684" y1="30.099" x2="8.89" y2="34.29" width="0" layer="19" extent="16-16"/>
+<contactref element="Q2" pad="TX"/>
+<wire x1="10.795" y1="28.575" x2="11.43" y2="29.21" width="0.4064" layer="16"/>
+<wire x1="11.43" y1="29.21" x2="12.7" y2="29.21" width="0.4064" layer="16"/>
+<wire x1="11.43" y1="29.21" x2="8.89" y2="34.29" width="0" layer="19" extent="16-16"/>
 </signal>
 <signal name="V+">
 <contactref element="U$2" pad="RAW"/>
-<contactref element="U$1" pad="12V-OUT"/>
-<wire x1="12.7" y1="34.671" x2="12.7" y2="35.56" width="0.4064" layer="16"/>
-<wire x1="12.7" y1="35.56" x2="11.43" y2="36.83" width="0.4064" layer="16"/>
-<wire x1="11.43" y1="36.83" x2="11.43" y2="38.1" width="0.4064" layer="16"/>
+<contactref element="Q2" pad="12V-OUT"/>
+<wire x1="11.43" y1="38.1" x2="11.43" y2="34.29" width="0.4064" layer="16"/>
+<wire x1="11.43" y1="34.29" x2="12.7" y2="33.02" width="0.4064" layer="16"/>
 </signal>
 <signal name="GND">
@@
 <contactref element="U$2" pad="GND1"/>
 <contactref element="U$2" pad="GND4"/>
-<contactref element="U$1" pad="GND"/>
-<contactref element="U$1" pad="GND"/>
 <contactref element="X1" pad="8"/>
 <contactref element="X1" pad="7"/>
@@
 <wire x1="48.43" y1="6.03" x2="47.94" y2="6.03" width="0.4064" layer="16"/>
 <wire x1="47.94" y1="6.03" x2="46.99" y2="5.08" width="0.4064" layer="16"/>
-<wire x1="52.2" y1="17.272" x2="43.35" y2="13.65" width="0" layer="19" extent="16-16"/>
+<contactref element="Q2" pad="GND"/>
+<contactref element="Q2" pad="GND"/>
+<wire x1="43.35" y1="13.65" x2="52.2" y2="17.272" width="0" layer="19" extent="16-16"/>
 </signal>
 <signal name="VCC">
 <contactref element="U$2" pad="VCC2"/>
 <contactref element="U$2" pad="VCC1"/>
-<contactref element="U$1" pad="5V-IN"/>
 <contactref element="Q1" pad="VCC"/>
 <contactref element="Q1" pad="VCC"/>
 <contactref element="SL2" pad="3"/>
 <wire x1="19.05" y1="38.1" x2="19.05" y2="36.83" width="0.4064" layer="16"/>
-<wire x1="19.05" y1="36.83" x2="15.24" y2="33.02" width="0.4064" layer="16"/>
-<wire x1="15.24" y1="33.02" x2="12.827" y2="33.02" width="0.4064" layer="16"/>
-<wire x1="12.827" y1="33.02" x2="12.7" y2="33.147" width="0.4064" layer="16"/>
+<wire x1="19.05" y1="36.83" x2="13.97" y2="31.75" width="0.4064" layer="16"/>
 <wire x1="45.72" y1="38.1" x2="44.45" y2="38.1" width="0.4064" layer="16"/>
 <wire x1="19.05" y1="3.81" x2="19.05" y2="7.62" width="0.4064" layer="16"/>
@@
 <wire x1="20.32" y1="35.56" x2="19.05" y2="36.83" width="0.4064" layer="16"/>
 <wire x1="25.4" y1="13.97" x2="25.4" y2="35.56" width="0.4064" layer="16"/>
-<wire x1="12.7" y1="33.147" x2="8.89" y2="29.21" width="0" layer="19" extent="1-1"/>
+<contactref element="Q2" pad="5V-IN"/>
+<wire x1="12.7" y1="31.75" x2="13.97" y2="31.75" width="0.4064" layer="16"/>
+<wire x1="12.7" y1="31.75" x2="8.89" y2="29.21" width="0" layer="19" extent="1-1"/>
 </signal>
 <signal name="N$7">
-<contactref element="U$1" pad="B"/>
 <contactref element="X1" pad="2"/>
 <wire x1="52.07" y1="22.225" x2="50.8" y2="22.225" width="0.4064" layer="16"/>
 <wire x1="50.8" y1="22.225" x2="49.53" y2="23.495" width="0.4064" layer="16"/>
-<wire x1="49.53" y1="23.495" x2="49.53" y2="29.21" width="0.4064" layer="16"/>
-<wire x1="36.83" y1="31.623" x2="47.117" y2="31.623" width="0.4064" layer="16"/>
-<wire x1="47.117" y1="31.623" x2="49.53" y2="29.21" width="0.4064" layer="16"/>
+<wire x1="49.53" y1="23.495" x2="49.53" y2="27.94" width="0.4064" layer="16"/>
+<wire x1="46.99" y1="30.48" x2="49.53" y2="27.94" width="0.4064" layer="16"/>
+<contactref element="Q2" pad="B"/>
+<wire x1="36.83" y1="30.48" x2="46.99" y2="30.48" width="0.4064" layer="16"/>
 </signal>
 <signal name="N$8">
-<contactref element="U$1" pad="A"/>
 <contactref element="X1" pad="1"/>
 <wire x1="54.61" y1="20.955" x2="53.975" y2="20.955" width="0.4064" layer="16"/>
@@
 <wire x1="53.34" y1="20.32" x2="49.53" y2="20.32" width="0.4064" layer="16"/>
 <wire x1="49.53" y1="20.32" x2="48.26" y2="21.59" width="0.4064" layer="16"/>
-<wire x1="48.26" y1="21.59" x2="48.26" y2="27.94" width="0.4064" layer="16"/>
-<wire x1="36.83" y1="30.099" x2="46.101" y2="30.099" width="0.4064" layer="16"/>
-<wire x1="46.101" y1="30.099" x2="48.26" y2="27.94" width="0.4064" layer="16"/>
+<wire x1="48.26" y1="21.59" x2="48.26" y2="26.67" width="0.4064" layer="16"/>
+<wire x1="45.72" y1="29.21" x2="48.26" y2="26.67" width="0.4064" layer="16"/>
+<contactref element="Q2" pad="A"/>
+<wire x1="36.83" y1="29.21" x2="45.72" y2="29.21" width="0.4064" layer="16"/>
 </signal>
 <signal name="N$9">
@@
 </signal>
 <signal name="N$5">
-<contactref element="U$1" pad="12V-IN"/>
 <contactref element="X1" pad="4"/>
 <contactref element="X1" pad="5"/>
 <contactref element="SL1" pad="1"/>
 <contactref element="SL3" pad="1"/>
-<wire x1="36.83" y1="28.575" x2="45.085" y2="28.575" width="0.4064" layer="16"/>
-<wire x1="45.085" y1="28.575" x2="46.99" y2="26.67" width="0.4064" layer="16"/>
-<wire x1="46.99" y1="26.67" x2="46.99" y2="17.145" width="0.4064" layer="16"/>
+<wire x1="44.45" y1="27.94" x2="46.99" y2="25.4" width="0.4064" layer="16"/>
+<wire x1="46.99" y1="25.4" x2="46.99" y2="17.145" width="0.4064" layer="16"/>
 <wire x1="46.99" y1="17.145" x2="49.53" y2="14.605" width="0.4064" layer="16"/>
 <wire x1="49.53" y1="14.605" x2="56.515" y2="14.605" width="0.4064" layer="16"/>
@@
 <wire x1="57.15" y1="12.7" x2="57.15" y2="13.97" width="0.8128" layer="16"/>
 <wire x1="57.15" y1="12.7" x2="57.15" y2="5.08" width="0.8128" layer="16"/>
+<contactref element="Q2" pad="12V-IN"/>
+<wire x1="36.83" y1="27.94" x2="44.45" y2="27.94" width="0.4064" layer="16"/>
 </signal>
 <signal name="D10">
