File: eagle/v1-controller.sch (EAGLE design)
At the start: 13 parts, among them Q1 DHT##, X1 RJ45-6L21-B

Commit message: Finished v1
Parts:
- removed U$1: RS485-ADAPTER, serge:RS485-ADAPTER
- added Q2: RS485-ADAPTER0.05-CONNECTOR, serge:RS485-ADAPTER0.05-CONNECTOR
Connections:
- net D2: now also Q2.RE/DE; no longer U$1.RE/DE
- net GND: now also Q2.GND; no longer U$1.GND
- net N$5: now also Q2.12V-IN; no longer U$1.12V-IN
- net N$7: now also Q2.B; no longer U$1.B
- net N$8: now also Q2.A; no longer U$1.A
- net RX: now also Q2.RX; no longer U$1.RX
- net TX: now also Q2.TX; no longer U$1.TX
- net V+: now also Q2.12V-OUT; no longer U$1.12V-OUT
- net VCC: now also Q2.5V-IN; no longer U$1.5V-IN
Changed lines of the file:
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@@
 <part name="P+3" library="supply1" deviceset="V+" device=""/>
 <part name="P+4" library="supply1" deviceset="VCC" device=""/>
-<part name="U$1" library="serge" deviceset="RS485-ADAPTER" device=""/>
 <part name="X1" library="con-tycoelectronics" deviceset="RJ45*2" device="1-B" technology="-6L"/>
 <part name="R1" library="adafruit" deviceset="R-US_" device="R0603" value="120"/>
@@
 <part name="SL3" library="con-amp-quick" deviceset="M02" device=""/>
 <part name="GND6" library="supply1" deviceset="GND" device=""/>
+<part name="Q2" library="serge" deviceset="RS485-ADAPTER" device="0.05-CONNECTOR"/>
 </parts>
 <sheets>
@@
 <instance part="P+3" gate="1" x="63.5" y="73.66" rot="R90"/>
 <instance part="P+4" gate="VCC" x="68.58" y="71.12" rot="R90"/>
-<instance part="U$1" gate="G$1" x="88.9" y="71.12"/>
 <instance part="X1" gate="G$1" x="137.16" y="60.96"/>
 <instance part="R1" gate="G$1" x="104.14" y="20.32"/>
@@
 <instance part="SL3" gate="G$1" x="175.26" y="38.1" rot="R180"/>
 <instance part="GND6" gate="1" x="165.1" y="10.16"/>
+<instance part="Q2" gate="G$1" x="88.9" y="71.12"/>
 </instances>
 <busses>
@@
 <net name="N$7" class="0">
 <segment>
-<pinref part="U$1" gate="G$1" pin="B"/>
 <pinref part="X1" gate="G$1" pin="2"/>
 <wire x1="129.54" y1="68.58" x2="106.68" y2="68.58" width="0.1524" layer="91"/>
+<pinref part="Q2" gate="G$1" pin="B"/>
 </segment>
 </net>
 <net name="N$8" class="0">
 <segment>
-<pinref part="U$1" gate="G$1" pin="A"/>
 <pinref part="X1" gate="G$1" pin="1"/>
 <wire x1="129.54" y1="71.12" x2="106.68" y2="71.12" width="0.1524" layer="91"/>
+<pinref part="Q2" gate="G$1" pin="A"/>
 </segment>
 </net>
@@
 <wire x1="81.28" y1="68.58" x2="76.2" y2="68.58" width="0.1524" layer="91"/>
 <label x="73.66" y="68.58" size="1.778" layer="95"/>
-<pinref part="U$1" gate="G$1" pin="RE/DE"/>
+<pinref part="Q2" gate="G$1" pin="RE/DE"/>
 </segment>
 </net>
@@
 <wire x1="81.28" y1="63.5" x2="76.2" y2="63.5" width="0.1524" layer="91"/>
 <label x="73.66" y="63.5" size="1.778" layer="95"/>
-<pinref part="U$1" gate="G$1" pin="RX"/>
+<pinref part="Q2" gate="G$1" pin="RX"/>
 </segment>
 </net>
@@
 <wire x1="81.28" y1="66.04" x2="76.2" y2="66.04" width="0.1524" layer="91"/>
 <label x="73.66" y="66.04" size="1.778" layer="95"/>
-<pinref part="U$1" gate="G$1" pin="TX"/>
+<pinref part="Q2" gate="G$1" pin="TX"/>
 </segment>
 </net>
@@
 <wire x1="81.28" y1="73.66" x2="66.04" y2="73.66" width="0.1524" layer="91"/>
 <pinref part="P+3" gate="1" pin="V+"/>
-<pinref part="U$1" gate="G$1" pin="12V-OUT"/>
+<pinref part="Q2" gate="G$1" pin="12V-OUT"/>
 </segment>
 </net>
@@
 <wire x1="111.76" y1="63.5" x2="111.76" y2="53.34" width="0.1524" layer="91"/>
 <pinref part="GND2" gate="1" pin="GND"/>
-<pinref part="U$1" gate="G$1" pin="GND"/>
 <pinref part="X1" gate="G$1" pin="8"/>
 <wire x1="111.76" y1="53.34" x2="111.76" y2="48.26" width="0.1524" layer="91"/>
@@
 <junction x="132.08" y="48.26"/>
 <junction x="129.54" y="53.34"/>
+<pinref part="Q2" gate="G$1" pin="GND"/>
 </segment>
 <segment>
@@
 <wire x1="81.28" y1="71.12" x2="71.12" y2="71.12" width="0.1524" layer="91"/>
 <pinref part="P+4" gate="VCC" pin="VCC"/>
-<pinref part="U$1" gate="G$1" pin="5V-IN"/>
+<pinref part="Q2" gate="G$1" pin="5V-IN"/>
 </segment>
 <segment>
@@
 <junction x="127" y="63.5"/>
 <wire x1="127" y1="73.66" x2="127" y2="63.5" width="0.1524" layer="91"/>
-<pinref part="U$1" gate="G$1" pin="12V-IN"/>
 <wire x1="106.68" y1="73.66" x2="127" y2="73.66" width="0.1524" layer="91"/>
 <pinref part="SL1" gate="G$1" pin="1"/>
@@
 <wire x1="147.32" y1="45.72" x2="121.92" y2="45.72" width="0.1524" layer="91"/>
 <junction x="121.92" y="45.72"/>
-</segment>
-</net>
+<pinref part="Q2" gate="G$1" pin="12V-IN"/>
+</segment>
+</net>
